File: MCU-LoRa.kicad_pcb (KiCad board)
At the start: 2 copper layers, 22.9 x 49 mm, 40 parts, among them J7 Conn_01x08_Pin, J8 Conn_01x08_Pin, J9 Conn_02x04_Top_Bottom, SW1 SW_Push, SW2 SW_Push, U1 RFM95W-915S2, U2 STM32F411CEU6, Y1 32.758kHz, Y2 25MHz

Commit message: ongoing cleanup. DRC clean excluding edge cut of castellated holes.
Parts:
- J7, J8: value Conn_01x08_Pin -> castellated_1x08_P2.54
Other:
- board text added: "(SCL2)B10"
- board text added: "A8"
- board text added: "A9"
- board text added: "B10"
- board text added: "B3"
- board text added: "B3(SDA2)"
- board text added: "B8"
- board text added: "B8(SCL1)"
- board text added: "B9"
- board text added: "B9(SDA1)"
- board text added: "VBAT"
- board text added: "v0.1.0 2025-10"
- board text removed: "a8"
- board text removed: "b8"
- board text removed: "b9"
- board text removed: "v0.1.0 2025-09"
Changed lines of the file:
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@@
 		)
 		(fp_text user "${REFERENCE}"
-			(at 0 3.5 180)
+			(at -3.124 0.096685 180)
 			(layer "F.Fab")
 			(effects
@@
 		)
 		(property "Value" "4.7µF"
-			(at 0 1.16 135)
+			(at 0.367696 2.305168 225)
 			(layer "F.Fab")
 			(effects
@@
 		(tags "resistor")
 		(property "Reference" "R12"
-			(at 12.92 3.93 0)
+			(at 1.26 -0.27 0)
 			(layer "F.SilkS")
+			(hide yes)
 			(effects
 				(font
@@
 			(at -0.551543 -1.205879 0)
 			(layer "F.Fab")
+			(hide yes)
 			(effects
 				(font
@@
 			)
 		)
-		(property "Value" "Conn_01x08_Pin"
+		(property "Value" "castellated_1x08_P2.54"
 			(at 0 -2.5 90)
 			(layer "F.Fab")
@@
 			)
 		)
-		(property "Datasheet" "~"
+		(property "Datasheet" ""
 			(at 0 0 90)
 			(layer "F.Fab")
@@
 			)
 		)
-		(property "Description" "Generic connector, single row, 01x08, script generated"
+		(property "Description" ""
 			(at 0 0 90)
 			(layer "F.Fab")
@@
 		(attr through_hole exclude_from_bom dnp)
 		(fp_line
-			(start 10.19 0.1016)
+			(start 10.19 0.254)
 			(end 10.19 1.5)
 			(stroke
@@
 		(fp_line
 			(start -10.19 1.5)
-			(end -10.19 0.1016)
+			(end -10.19 0.254)
 			(stroke
 				(width 0.12)
@@
 		)
 		(fp_line
-			(start 9.94 0.0508)
+			(start 9.94 -1.25)
 			(end 9.94 1.25)
 			(stroke
@@
 		)
 		(fp_line
+			(start -9.94 -1.25)
+			(end 9.94 -1.25)
+			(stroke
+				(width 0.05)
+				(type default)
+			)
+			(layer "F.CrtYd")
+		)
+		(fp_line
 			(start 9.94 1.25)
 			(end -9.94 1.25)
@@
 		(fp_line
 			(start -9.94 1.25)
-			(end -9.94 0.0508)
+			(end -9.94 -1.25)
 			(stroke
 				(width 0.05)
@@
 		)
 		(property "Value" "STM32F411CEU6"
-			(at 0 4.83 315)
+			(at -0.106173 1.88794 180)
 			(layer "F.Fab")
 			(effects
@@
 		(tags "inductor")
 		(property "Reference" "L1"
-			(at 0.256359 10.52 90)
+			(at 0.54 0.51 90)
 			(layer "F.SilkS")
+			(hide yes)
 			(effects
 				(font
@@
 			(at 0 1.17 90)
 			(layer "F.Fab")
+			(hide yes)
 			(effects
 				(font
@@
 			)
 		)
-		(property "Value" "Conn_01x08_Pin"
+		(property "Value" "castellated_1x08_P2.54"
 			(at 0.21 -2.68 90)
 			(layer "F.Fab")
@@
 			)
 		)
-		(property "Datasheet" "~"
+		(property "Datasheet" ""
 			(at 0 0 90)
 			(layer "F.Fab")
@@
 			)
 		)
-		(property "Description" "Generic connector, single row, 01x08, script generated"
+		(property "Description" ""
 			(at 0 0 90)
 			(layer "F.Fab")
@@
 		(fp_line
 			(start -10.19 1.5)
-			(end -10.19 0.1016)
+			(end -10.19 0.254)
 			(stroke
 				(width 0.12)
@@
 		)
 		(fp_line
-			(start 10.19 0.1016)
+			(start 10.19 0.254)
 			(end 10.19 1.5)
 			(stroke
@@
 		(fp_line
 			(start -9.94 1.25)
-			(end -9.94 0.0508)
+			(end -9.94 -1.25)
 			(stroke
 				(width 0.05)
@@
 		)
 		(fp_line
-			(start 9.94 0.0508)
+			(start -9.94 -1.25)
+			(end 9.94 -1.25)
+			(stroke
+				(width 0.05)
+				(type default)
+			)
+			(layer "F.CrtYd")
+		)
+		(fp_line
+			(start 9.94 -1.25)
 			(end 9.94 1.25)
 			(stroke
@@
 		(tags "capacitor")
 		(property "Reference" "C7"
-			(at 5.87 -15.12 90)
+			(at 0.01 -0.81 90)
 			(layer "F.SilkS")
+			(hide yes)
 			(effects
 				(font
@@
 			(at 0 1.16 90)
 			(layer "F.Fab")
+			(hide yes)
 			(effects
 				(font
@@
 			)
 		)
-		(property "Silk2" "b2"
+		(property "Silk2" "B2"
 			(at -2.222 -0.784 0)
 			(unlocked yes)
@@
 			(effects
 				(font
-					(size 1 1)
-					(thickness 0.15)
+					(size 0.8 0.8)
+					(thickness 0.1)
 				)
 			)
@@
 		(layer "Edge.Cuts")
 	)
-	(gr_text "a8"
-		(at 35.512 60.512 0)
+	(gr_text "A8"
+		(at 62.67 71.19 0)
 		(layer "F.SilkS")
 		(effects
 			(font
-				(size 1 1)
-				(thickness 0.15)
+				(size 0.8 0.8)
+				(thickness 0.1)
+			)
+			(justify left bottom)
+		)
+	)
+	(gr_text "B8"
+		(at 70.75 58.51 90)
+		(layer "F.SilkS")
+		(effects
+			(font
+				(size 0.8 0.8)
+				(thickness 0.1)
 			)
 			(justify left bottom)
@@
 		)
 	)
-	(gr_text "v0.1.0 2025-09"
+	(gr_text "VBAT"
+		(at 70.71 61.6 90)
+		(layer "F.SilkS")
+		(effects
+			(font
+				(size 0.8 0.8)
+				(thickness 0.1)
+			)
+			(justify left bottom)
+		)
+	)
+	(gr_text "v0.1.0 2025-10"
 		(at 51.006 94.802 0)
 		(layer "F.SilkS")
@@
 		)
 	)
+	(gr_text "B9"
+		(at 70.75 56.14 90)
+		(layer "F.SilkS")
+		(effects
+			(font
+				(size 0.8 0.8)
+				(thickness 0.1)
+			)
+			(justify left bottom)
+		)
+	)
+	(gr_text "B3"
+		(at 70.78 66.27 90)
+		(layer "F.SilkS")
+		(effects
+			(font
+				(size 0.8 0.8)
+				(thickness 0.1)
+			)
+			(justify left bottom)
+		)
+	)
 	(gr_text "F411-RFM95W"
 		(at 50.498 93.024 0)
@@
 		)
 	)
-	(gr_text "b8"
-		(at 43.16 63.8 0)
+	(gr_text "SLC1"
+		(at 61.95 56.61 0)
 		(layer "F.SilkS")
 		(effects
@@
 		)
 	)
-	(gr_text "SLC1"
-		(at 62.179881 56.498002 0)
+	(gr_text "A9"
+		(at 70.79 68.96 90)
 		(layer "F.SilkS")
 		(effects
@@
 		)
 	)
-	(gr_text "b9"
-		(at 41.53 72.82 0)
+	(gr_text "3v3"
+		(at 65.25 47.45 0)
 		(layer "F.SilkS")
 		(effects
@@
 		)
 	)
-	(gr_text "3v3"
-		(at 65.25 47.45 0)
+	(gr_text "GND"
+		(at 56.85 56.76 0)
 		(layer "F.SilkS")
 		(effects
@@
 		)
 	)
-	(gr_text "GND"
-		(at 58.03 56.702 90)
+	(gr_text "B10"
+		(at 51.32 61.84 270)
 		(layer "F.SilkS")
 		(effects
@@
 		)
 	)
+	(gr_text "A9"
+		(at 70.93 68.56 0)
+		(layer "B.SilkS")
+		(effects
+			(font
+				(size 0.8 0.8)
+				(thickness 0.1)
+			)
+			(justify left bottom mirror)
+		)
+	)
+	(gr_text "(SCL2)B10"
+		(at 57.17 63.39 0)
+		(layer "B.SilkS")
+		(effects
+			(font
+				(size 0.8 0.8)
+				(thickness 0.1)
+			)
+			(justify left bottom mirror)
+		)
+	)
+	(gr_text "B8(SCL1)"
+		(at 70.95 58.49 0)
+		(layer "B.SilkS")
+		(effects
+			(font
+				(size 0.8 0.8)
+				(thickness 0.1)
+			)
+			(justify left bottom mirror)
+		)
+	)
+	(gr_text "B9(SDA1)"
+		(at 70.97 55.79 0)
+		(layer "B.SilkS")
+		(effects
+			(font
+				(size 0.8 0.8)
+				(thickness 0.1)
+			)
+			(justify left bottom mirror)
+		)
+	)
+	(gr_text "B3(SDA2)"
+		(at 70.82 66.06 0)
+		(layer "B.SilkS")
+		(effects
+			(font
+				(size 0.8 0.8)
+				(thickness 0.1)
+			)
+			(justify left bottom mirror)
+		)
+	)
 	(gr_text "3v3"
 		(at 52.96 65.89 0)
 		(layer "B.SilkS")
 		(effects
+			(font
+				(size 0.8 0.8)
+				(thickness 0.1)
+			)
+			(justify left bottom mirror)
+		)
+	)
+	(gr_text "VBAT"
+		(at 70.87 60.95 0)
+		(layer "B.SilkS")
+		(effects

Commit message: ongoing
Other:
- board text added: "(SCL2)PB10"
- board text added: "PA9"
- board text added: "PB3(SDA2)"
- board text added: "PB8(SCL1)"
- board text added: "PB9(SDA1)"
- board text added: "led PC13"
- board text removed: "(SCL2)B10"
- board text removed: "B3(SDA2)"
- board text removed: "B8(SCL1)"
- board text removed: "B9(SDA1)"
Changed lines of the file:
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@@
 		)
 	)
-	(gr_text "A9"
+	(gr_text "PA9"
 		(at 70.93 68.56 0)
 		(layer "B.SilkS")
@@
 		)
 	)
-	(gr_text "(SCL2)B10"
+	(gr_text "(SCL2)PB10"
 		(at 57.17 63.39 0)
 		(layer "B.SilkS")
@@
 		)
 	)
-	(gr_text "B8(SCL1)"
+	(gr_text "PB8(SCL1)"
 		(at 70.95 58.49 0)
 		(layer "B.SilkS")
@@
 		)
 	)
-	(gr_text "B9(SDA1)"
+	(gr_text "PB9(SDA1)"
 		(at 70.97 55.79 0)
 		(layer "B.SilkS")
@@
 		)
 	)
-	(gr_text "B3(SDA2)"
+	(gr_text "PB3(SDA2)"
 		(at 70.82 66.06 0)
 		(layer "B.SilkS")
@@
 			)
 			(justify left bottom mirror)
+		)
+	)
+	(gr_text "led PC13"
+		(at 64.96 70.87 0)
+		(layer "B.SilkS")
+		(effects
+			(font
+				(size 1 1)
+			)
+			(justify left bottom mirror)
